Commit message: vx01.urdf.xacro main added

File: vx01_ws/src/vx01_description/urdf/drone/control/drone.ros2_control.xacro (robot description, xacro)
@@ -5,5 +5,6 @@
         prefix
         use_sim:=false
-        pwm_frequency:=50">
+        pwm_frequency:=50
+        gpio_chip:=gpiochip0">
         <ros2_control name="${name}" type="system">
             <!-- HARDWARE PLUGIN          -->
@@ -17,13 +18,9 @@
                     <plugin>vx01_drone_hardware/DroneHardwareInterface</plugin>
                     <param name="pwm_frequency">${pwm_frequency}</param>
-                    <!-- GPIO pins for arm servos on RDK X5 -->
-                    <param name="arm_servo_0_pin">20</param>
-                    <param name="arm_servo_1_pin">21</param>
-                    <param name="arm_servo_2_pin">22</param>
-                    <param name="arm_servo_3_pin">23</param>
+                    <param name="gpio_chip">${gpio_chip}</param>
                 </xacro:unless>
             </hardware>
-            <!-- ARM 0 - Roll axis servo -->
-            <joint name="${prefix}drone_arm0_joint">
+            <!-- ARM 0 - Roll axis servo (matches arm_joint0 in URDF) -->
+            <joint name="${prefix}arm_joint0">
                 <command_interface name="position">
                     <param name="min">-1.5707963</param>
@@ -42,14 +39,14 @@
                 <param name="reversed">false</param>
             </joint>
-            <!-- ARM 1 -->
-            <joint name="${prefix}drone_arm1_joint">
+            <!-- ARM 1 (matches arm_joint1 in URDF) -->
+            <joint name="${prefix}arm_joint1">
                 <command_interface name="position">
                     <param name="min">-1.5707963</param>
                     <param name="max">1.5707963</param>
                 </command_interface>
-                    <state_interface name="position">
-                        <param name="initial_value">0.0</param>
-                    </state_interface>
-                    <state_interface name="velocity"/>
+                <state_interface name="position">
+                    <param name="initial_value">0.0</param>
+                </state_interface>
+                <state_interface name="velocity"/>
                 <param name="gpio_pin">21</param>
                 <param name="min_pulse_us">500.0</param>
@@ -60,6 +57,6 @@
                 <param name="reversed">false</param>
             </joint>
-            <!-- ARM 2 -->
-            <joint name="${prefix}drone_arm2_joint">
+            <!-- ARM 2 (matches arm_joint2 in URDF) -->
+            <joint name="${prefix}arm_joint2">
                 <command_interface name="position">
                     <param name="min">-1.5707963</param>
@@ -78,6 +75,6 @@
                 <param name="reversed">false</param>
             </joint>
-            <!-- ARM 3 -->
-            <joint name="${prefix}drone_arm3_joint">
+            <!-- ARM 3 (matches arm_joint3 in URDF) -->
+            <joint name="${prefix}arm_joint3">
                 <command_interface name="position">
                     <param name="min">-1.5707963</param>

File: vx01_ws/src/vx01_description/urdf/hexapod/control/hexapod.ros2_control.xacro (robot description, xacro)
@@ -9,7 +9,4 @@
         <ros2_control name="${name}" type="system">
             <!-- Hardware Plugin -->
-            <buildtool_depend>rosidl_default_generators</buildtool_depend>
-            <depend>action_msgs</depend>
-            <member_of_group>rosidl_interface_packages</member_of_group>
             <hardware>
                 <xacro:if value="${use_sim}">
@@ -22,5 +19,5 @@
                 </xacro:unless>
             </hardware>
-            <!-- LEG 0 JOINTS  -->
+            <!-- LEG 0 JOINTS (Right Front) -->
             <joint name="${prefix}coxa_leg0_joint">
                 <command_interface name="position">
@@ -33,5 +30,4 @@
                 <state_interface name="velocity"/>
                 <state_interface name="effort"/>
-                <!-- Servo hardware params -->
                 <param name="servo_id">0</param>
                 <param name="min_pulse">500.0</param>
@@ -84,5 +80,5 @@
                 <param name="max_acceleration">20.0</param>
             </joint>
-            <!-- LEG 1 JOINTS -->
+            <!-- LEG 1 JOINTS (Right Middle) -->
             <joint name="${prefix}coxa_leg1_joint">
                 <command_interface name="position">
@@ -145,5 +141,5 @@
                 <param name="max_acceleration">20.0</param>
             </joint>
-            <!-- LEG 2 JOINTS -->
+            <!-- LEG 2 JOINTS (Right Rear) -->
             <joint name="${prefix}coxa_leg2_joint">
                 <command_interface name="position">
@@ -206,5 +202,5 @@
                 <param name="max_acceleration">20.0</param>
             </joint>
-            <!-- LEG 3 JOINTS (Left side) -->
+            <!-- LEG 3 JOINTS (Left Rear - reversed) -->
             <joint name="${prefix}coxa_leg3_joint">
                 <command_interface name="position">
@@ -267,5 +263,5 @@
                 <param name="max_acceleration">20.0</param>
             </joint>
-            <!-- LEG 4 JOINTS  -->
+            <!-- LEG 4 JOINTS (Left Middle - reversed) -->
             <joint name="${prefix}coxa_leg4_joint">
                 <command_interface name="position">
@@ -328,5 +324,5 @@
                 <param name="max_acceleration">20.0</param>
             </joint>
-            <!-- LEG 5 JOINTS -->
+            <!-- LEG 5 JOINTS (Left Front - reversed) -->
             <joint name="${prefix}coxa_leg5_joint">
                 <command_interface name="position">
