Commit message: robot loaded in gazebo

File: vx01_ws/src/vx01_description/urdf/sensors/imu.xacro (robot description, xacro)
@@ -1,53 +1,151 @@
 <?xml version="1.0"?>
 <robot xmlns:xacro="http://www.ros.org/wiki/xacro">
+    <!--
+        Hiwonder IM10A — 10-axis AHRS/INS IMU
+        ─────────────────────────────────────────────────────────────────
+        Accelerometer  : ±16g,  RMS noise 0.75 mg-rms @ 100Hz BW
+                         Zero drift ±20–40 mg,  Temp drift ±0.15 mg/°C
+        Gyroscope      : ±2000°/s, RMS noise 0.028–0.07 °/s-rms @ 100Hz
+                         Zero drift ±0.5–1 °/s, Temp drift ±0.005–0.015 °/s/°C
+        Magnetometer   : ±2 Gauss, 0.0667 mGauss/LSB
+        Barometer      : 300–1100 hPa, RMS noise 0.5 Pa
+        Output rate    : 10 Hz default, up to 200 Hz
+        Interface      : UART (9600–921600 bps) / I2C (up to 400 kHz)
+        Voltage        : 5V or 3.3V  |  Current: 12 mA
+        Noise conversions used for Gazebo:
+          Accel stddev  = 0.75e-3 g × 9.81        = 0.007358 m/s²
+          Accel bias    = 30e-3 g × 9.81 (mid)    = 0.2943  m/s²  ← zero drift mid
+          Gyro stddev   = 0.049 °/s × π/180       = 0.000855 rad/s  (mid of 0.028–0.07)
+          Gyro bias     = 0.75 °/s × π/180 (mid)  = 0.01309  rad/s  ← zero drift mid
+    -->
     <link name="imu_link">
         <inertial>
-            <origin
-                xyz="-4.9599E-19 -9.0896E-20 0.005"
-                rpy="0 0 0" />
-            <mass
-                value="0.0045937" />
+            <origin xyz="-4.9599E-19 -9.0896E-20 0.005" rpy="0 0 0"/>
+            <mass value="0.0045937"/>
             <inertia
-                ixx="1.9002E-07"
-                ixy="1.1915E-23"
-                ixz="5.4526E-24"
-                iyy="2.7817E-07"
-                iyz="-4.039E-25"
-                izz="3.9603E-07" />
+                ixx="1.9002E-07" ixy="1.1915E-23" ixz="5.4526E-24"
+                iyy="2.7817E-07" iyz="-4.039E-25"
+                izz="3.9603E-07"/>
         </inertial>
         <visual>
-            <origin
-                xyz="0 0 0"
-                rpy="0 0 0" />
+            <origin xyz="0 0 0" rpy="0 0 0"/>
             <geometry>
-                <mesh
-                    filename="package://vx01_description/meshes/sensors/imu_link.STL" />
+                <mesh filename="package://vx01_description/meshes/sensors/imu_link.STL"/>
             </geometry>
-            <material
-                name="">
-                <color
-                    rgba="0.79216 0.81961 0.93333 1" />
+            <material name="">
+                <color rgba="0.79216 0.81961 0.93333 1"/>
             </material>
         </visual>
         <collision>
-            <origin
-                xyz="0 0 0"
-                rpy="0 0 0" />
+            <origin xyz="0 0 0" rpy="0 0 0"/>
             <geometry>
-                <mesh
-                    filename="package://vx01_description/meshes/sensors/imu_link.STL" />
+                <mesh filename="package://vx01_description/meshes/sensors/imu_link.STL"/>
             </geometry>
         </collision>
     </link>
     <joint name="imu_joint" type="fixed">
-        <origin
-            xyz="-0.0013383 0 0.0025"
-            rpy="0 0 0" />
-        <parent
-            link="base_link" />
-        <child
-            link="imu_link" />
-        <axis
-            xyz="0 0 0" />
+        <origin xyz="-0.0013383 0 0.0025" rpy="0 0 0"/>
+        <parent link="base_link"/>
+        <child  link="imu_link"/>
+        <axis xyz="0 0 0"/>
     </joint>
+    <!-- ══════════════════════════════════════════════════════════════════
+         Ignition Gazebo IMU sensor — Hiwonder IM10A
+         Topic published: /imu/data  (sensor_msgs/msg/Imu)
+         ══════════════════════════════════════════════════════════════════ -->
+    <gazebo reference="imu_link">
+        <sensor name="imu_sensor" type="imu">
+            <ignition_frame_id>imu_link</ignition_frame_id>
+            <always_on>1</always_on>
+            <!-- IM10A: up to 200 Hz; 100 Hz is the practical sim rate -->
+            <update_rate>100</update_rate>
+            <visualize>false</visualize>
+            <topic>imu/data</topic>
+            <imu>
+                <!-- Orientation is fused on the real hardware by the Kalman filter.
+                     In sim we let the EKF node do it, so disable built-in orientation. -->
+                <enable_orientation>0</enable_orientation>
+                <!-- ── Gyroscope (IM10A: ±2000°/s, 0.028–0.07 °/s-rms noise) ── -->
+                <angular_velocity>
+                    <x>
+                        <noise type="gaussian">
+                            <mean>0.0</mean>
+                            <!-- RMS noise mid: 0.049 °/s = 0.000855 rad/s -->
+                            <stddev>0.000855</stddev>
+                            <!-- Zero drift mid: 0.75 °/s = 0.01309 rad/s -->
+                            <bias_mean>0.01309</bias_mean>
+                            <!-- Temp drift: 0.01 °/s/°C = 0.000175 rad/s/°C -->
+                            <bias_stddev>0.000175</bias_stddev>
+                            <dynamic_bias_stddev>0.000175</dynamic_bias_stddev>
+                            <dynamic_bias_correlation_time>400.0</dynamic_bias_correlation_time>
+                            <!-- Resolution: 0.061 (°/s)/LSB = 0.001065 rad/s -->
+                            <precision>0.001065</precision>
+                        </noise>
+                    </x>
+                    <y>
+                        <noise type="gaussian">
+                            <mean>0.0</mean>
+                            <stddev>0.000855</stddev>
+                            <bias_mean>0.01309</bias_mean>
+                            <bias_stddev>0.000175</bias_stddev>
+                            <dynamic_bias_stddev>0.000175</dynamic_bias_stddev>
+                            <dynamic_bias_correlation_time>400.0</dynamic_bias_correlation_time>
+                            <precision>0.001065</precision>
+                        </noise>
+                    </y>
+                    <z>
+                        <noise type="gaussian">
+                            <mean>0.0</mean>
+                            <stddev>0.000855</stddev>
+                            <bias_mean>0.01309</bias_mean>
+                            <bias_stddev>0.000175</bias_stddev>
+                            <dynamic_bias_stddev>0.000175</dynamic_bias_stddev>
+                            <dynamic_bias_correlation_time>400.0</dynamic_bias_correlation_time>
+                            <precision>0.001065</precision>
+                        </noise>
+                    </z>
+                </angular_velocity>
+                <!-- ── Accelerometer (IM10A: ±16g, 0.75 mg-rms noise) ── -->
+                <linear_acceleration>
+                    <x>
+                        <noise type="gaussian">
+                            <mean>0.0</mean>
+                            <!-- RMS noise: 0.75 mg × 9.81 = 0.007358 m/s² -->
+                            <stddev>0.007358</stddev>
+                            <!-- Zero drift mid: 30 mg × 9.81 = 0.2943 m/s² -->
+                            <bias_mean>0.2943</bias_mean>
+                            <!-- Temp drift: 0.15 mg/°C × 9.81 = 0.001472 m/s²/°C -->
+                            <bias_stddev>0.001472</bias_stddev>
+                            <dynamic_bias_stddev>0.001472</dynamic_bias_stddev>
+                            <dynamic_bias_correlation_time>175.0</dynamic_bias_correlation_time>
+                            <!-- Resolution: 0.0005 g/LSB × 9.81 = 0.004905 m/s² -->
+                            <precision>0.004905</precision>
+                        </noise>
+                    </x>
+                    <y>
+                        <noise type="gaussian">
+                            <mean>0.0</mean>
+                            <stddev>0.007358</stddev>
+                            <bias_mean>0.2943</bias_mean>
+                            <bias_stddev>0.001472</bias_stddev>
+                            <dynamic_bias_stddev>0.001472</dynamic_bias_stddev>
+                            <dynamic_bias_correlation_time>175.0</dynamic_bias_correlation_time>
+                            <precision>0.004905</precision>
+                        </noise>
+                    </y>
+                    <z>
+                        <noise type="gaussian">
+                            <mean>0.0</mean>
+                            <stddev>0.007358</stddev>
+                            <bias_mean>0.2943</bias_mean>
+                            <bias_stddev>0.001472</bias_stddev>
+                            <dynamic_bias_stddev>0.001472</dynamic_bias_stddev>
+                            <dynamic_bias_correlation_time>175.0</dynamic_bias_correlation_time>
+                            <precision>0.004905</precision>
+                        </noise>
+                    </z>
+                </linear_acceleration>
+            </imu>
+        </sensor>
+    </gazebo>
 </robot>

File: vx01_ws/src/vx01_description/urdf/sensors/tf_lidar.xacro (robot description, xacro)
@@ -1,53 +1,98 @@
 <?xml version="1.0"?>
 <robot xmlns:xacro="http://www.ros.org/wiki/xacro">
+    <!--
+        Benewake TFmini-S — Single-point ToF LiDAR
+        ─────────────────────────────────────────────────────────────────
+        Range      : 0.1 m – 12 m @ 90% reflectivity
+                     0.1 m –  7 m @ 10% reflectivity (low reflectivity)
+        Accuracy   : ±6 cm  (0.1–6 m)  |  ±1%  (6–12 m)
+        Resolution : 1 cm  (0.01 m)
+        FoV        : 2° (single-point — modelled as 2°×2° ray)
+        Frame rate : 1–1000 Hz  (default 100 Hz)
+        Wavelength : 850 nm VCSEL
+        Interface  : UART 115200 bps (default) / I²C
+        Voltage    : 5V ± 0.1V  |  Current ≤ 140 mA  |  Power ≤ 0.7 W
+        Size       : 42 × 15 × 16 mm  |  Weight: 5 g
+        Noise derivation:
+          Accuracy ±6 cm means 99.7% (3σ) of readings are within ±6 cm
+          → stddev = 0.06 / 3 = 0.02 m
+    -->
     <link name="lidar_link">
         <inertial>
-            <origin
-                xyz="-0.010087 0.00016968 8.5648E-05"
-                rpy="0 0 0" />
-            <mass
-                value="0.0060491" />
+            <origin xyz="-0.010087 0.00016968 8.5648E-05" rpy="0 0 0"/>
+            <mass value="0.0060491"/>
             <inertia
-                ixx="6.6215E-07"
-                ixy="4.0559E-09"
-                ixz="2.4269E-09"
-                iyy="1.8783E-07"
-                iyz="-4.799E-11"
-                izz="6.474E-07" />
+                ixx="6.6215E-07" ixy="4.0559E-09" ixz="2.4269E-09"
+                iyy="1.8783E-07" iyz="-4.799E-11"
+                izz="6.474E-07"/>
         </inertial>
         <visual>
-            <origin
-                xyz="0 0 0"
-                rpy="0 0 0" />
+            <origin xyz="0 0 0" rpy="0 0 0"/>
             <geometry>
-                <mesh
-                    filename="package://vx01_description/meshes/sensors/lidar_link.STL" />
+                <mesh filename="package://vx01_description/meshes/sensors/lidar_link.STL"/>
             </geometry>
-            <material
-                name="">
-                <color
-                    rgba="0.29804 0.29804 0.29804 1" />
+            <material name="">
+                <color rgba="0.29804 0.29804 0.29804 1"/>
             </material>
         </visual>
         <collision>
-            <origin
-                xyz="0 0 0"
-                rpy="0 0 0" />
+            <origin xyz="0 0 0" rpy="0 0 0"/>
             <geometry>
-                <mesh
-                    filename="package://vx01_description/meshes/sensors/lidar_link.STL" />
+                <mesh filename="package://vx01_description/meshes/sensors/lidar_link.STL"/>
             </geometry>
         </collision>
     </link>
+    <!-- Sensor faces forward (X axis) via 90° pitch rotation -->
     <joint name="lidar_joint" type="fixed">
-        <origin
-            xyz="-0.070325 -0.00034592 0"
-            rpy="0.0057344 1.5708 0" />
-        <parent
-            link="base_link" />
-        <child
-            link="lidar_link" />
-        <axis
-            xyz="0 0 0" />
+        <origin xyz="-0.070325 -0.00034592 0" rpy="0.0057344 1.5708 0"/>
+        <parent link="base_link"/>
+        <child  link="lidar_link"/>
+        <axis xyz="0 0 0"/>
     </joint>
+    <!-- ══════════════════════════════════════════════════════════════════
+         Ignition Gazebo GPU Ray sensor — Benewake TFmini-S
+         type="gpu_ray"  ← correct for Ignition Fortress (not gpu_lidar)
+         Single-point modelled as a 2°×2° ray fan (1×1 sample).
+         Publishes: sensor_msgs/msg/LaserScan on /lidar/scan
+         ══════════════════════════════════════════════════════════════════ -->
+    <gazebo reference="lidar_link">
+        <sensor name="tfmini_s" type="gpu_ray">
+            <ignition_frame_id>lidar_link</ignition_frame_id>
+            <always_on>1</always_on>
+            <!-- TFmini-S default frame rate: 100 Hz -->
+            <update_rate>100</update_rate>
+            <visualize>false</visualize>
+            <topic>lidar/scan</topic>
+            <ray>
+                <scan>
+                    <!-- 1 sample spanning the full 2° (0.03491 rad) beam -->
+                    <horizontal>
+                        <samples>1</samples>
+                        <resolution>1</resolution>
+                        <min_angle>-0.01745</min_angle>  <!-- -1° -->
+                        <max_angle>0.01745</max_angle>   <!-- +1° -->
+                    </horizontal>
+                    <vertical>
+                        <samples>1</samples>
+                        <resolution>1</resolution>
+                        <min_angle>-0.01745</min_angle>  <!-- -1° -->
+                        <max_angle>0.01745</max_angle>   <!-- +1° -->
+                    </vertical>
+                </scan>
+                <range>
+                    <!-- TFmini-S: 0.1 m min blind-zone end, 12 m max -->
+                    <min>0.1</min>
+                    <max>12.0</max>
+                    <!-- Datasheet resolution: 1 cm -->
+                    <resolution>0.01</resolution>
+                </range>
+                <noise>
+                    <type>gaussian</type>
+                    <mean>0.0</mean>
+                    <!-- ±6 cm accuracy @ 3σ → stddev = 0.06/3 = 0.02 m -->
+                    <stddev>0.02</stddev>
+                </noise>
+            </ray>
+        </sensor>
+    </gazebo>
 </robot>

File: vx01_ws/src/vx01_description/urdf/vx01.urdf.xacro (robot description, xacro)
@@ -1,10 +1,11 @@
 <?xml version="1.0"?>
 <robot name="vx01" xmlns:xacro="http://www.ros.org/wiki/xacro">
-    <!-- PROPERTIES -->
-    <xacro:property name="use_sim" value="false"/>
-    <xacro:property name="prefix" value=""/>
-    <!-- Base body -->
+    <xacro:arg name="use_sim" default="false"/>
+    <xacro:property name="use_sim" value="$(arg use_sim)"/>
+    <xacro:arg name="prefix" default=""/>
+    <xacro:property name="prefix" value="$(arg prefix)"/>
+    <!-- ── Base body ── -->
     <xacro:include filename="$(find vx01_description)/urdf/base/base.xacro"/>
-    <!-- Hexapod legs (6 legs) -->
+    <!-- ── Hexapod legs (6 legs) ── -->
     <xacro:include filename="$(find vx01_description)/urdf/hexapod/leg_0.xacro"/>
     <xacro:include filename="$(find vx01_description)/urdf/hexapod/leg_1.xacro"/>
@@ -13,67 +14,31 @@
     <xacro:include filename="$(find vx01_description)/urdf/hexapod/leg_4.xacro"/>
     <xacro:include filename="$(find vx01_description)/urdf/hexapod/leg_5.xacro"/>
-    <!-- Drone arms (4 arms with props) -->
+    <!-- ── Drone arms (4 arms with props) ── -->
     <xacro:include filename="$(find vx01_description)/urdf/drone/arm_0.xacro"/>
     <xacro:include filename="$(find vx01_description)/urdf/drone/arm_1.xacro"/>
     <xacro:include filename="$(find vx01_description)/urdf/drone/arm_2.xacro"/>
     <xacro:include filename="$(find vx01_description)/urdf/drone/arm_3.xacro"/>
-    <!-- Sensors -->
+    <!-- ── Sensors ── -->
     <xacro:include filename="$(find vx01_description)/urdf/sensors/depth_camera.xacro"/>
     <xacro:include filename="$(find vx01_description)/urdf/sensors/imu.xacro"/>
     <xacro:include filename="$(find vx01_description)/urdf/sensors/tf_lidar.xacro"/>
-    <!-- ROS2 Control interfaces -->
-    <xacro:include filename="$(find vx01_description)/urdf/hexapod/control/hexapod.ros2_control.xacro"/>
-    <xacro:include filename="$(find vx01_description)/urdf/drone/control/drone.ros2_control.xacro"/>
-    <!-- Hexapod control (18 servo joints) -->
-    <xacro:hexapod_ros2_control
-        name="hexapod_controller"
+    <!-- ROS2_control -->
+    <xacro:include filename="$(find vx01_description)/urdf/control/vx01.ros2_control.xacro"/>
+    <!-- Gazebo reference -->
+    <xacro:include filename="$(find vx01_description)/urdf/gazebo/vx01_sim.xacro"/>
+    <xacro:vx01_ros2_control
         prefix="${prefix}"
         use_sim="${use_sim}"
         serial_port="/dev/ttyACM0"
-        baud_rate="115200"/>
-    <!-- Drone arm control (4 servo joints via GPIO) -->
-    <xacro:drone_ros2_control
-        name="drone_controller"
-        prefix="${prefix}"
-        use_sim="${use_sim}"
+        baud_rate="115200"
         pwm_frequency="50"
         gpio_chip="gpiochip0"/>
-    <!-- GAZEBO PLUGINS (for simulation)            -->
+    <!-- Gazebo / Ignition Fortress Simulation Plugins -->
     <xacro:if value="${use_sim}">
-        <!-- Gazebo ROS2 Control plugin -->
         <gazebo>
-            <plugin filename="libgazebo_ros2_control.so" name="gazebo_ros2_control">
-                <robot_param>robot_description</robot_param>
-                <robot_param_node>robot_state_publisher</robot_param_node>
-                <parameters>$(find vx01_bringup)/config/hexapod/controller_manager.yaml</parameters>
-                <parameters>$(find vx01_bringup)/config/drone/controller_manager.yaml</parameters>
+            <plugin filename="gz_ros2_control-system" name="gz_ros2_control::GazeboSimROS2ControlPlugin">
+                <parameters>$(find vx01_bringup)/config/vx01_controller_manager.yaml</parameters>
             </plugin>
         </gazebo>
-        <!-- Ground plane contact -->
-        <gazebo reference="base_link">
-            <mu1>0.8</mu1>
-            <mu2>0.8</mu2>
-            <kp>1000000.0</kp>
-            <kd>100.0</kd>
-            <minDepth>0.001</minDepth>
-            <maxVel>1.0</maxVel>
-        </gazebo>
-        <!-- Leg tip contacts -->
-        <xacro:macro name="leg_contact" params="leg_num">
-            <gazebo reference="tibia_link_${leg_num}">
-                <mu1>1.0</mu1>
-                <mu2>1.0</mu2>
-                <kp>1000000.0</kp>
-                <kd>100.0</kd>
-                <minDepth>0.001</minDepth>
-                <maxVel>1.0</maxVel>
-            </gazebo>
-        </xacro:macro>
-        <xacro:leg_contact leg_num="0"/>
-        <xacro:leg_contact leg_num="1"/>
-        <xacro:leg_contact leg_num="2"/>
-        <xacro:leg_contact leg_num="3"/>
-        <xacro:leg_contact leg_num="4"/>
-        <xacro:leg_contact leg_num="5"/>
     </xacro:if>
 </robot>
