Commit message: fix: remove propeller collision meshes to resolve physics engine instability

File: vx01_ws/src/vx01_description/urdf/drone/arm_0.xacro (robot description, xacro)
@@ -135,13 +135,5 @@
             </material>
         </visual>
-        <collision>
-            <origin
-                xyz="0 0 0"
-                rpy="0 0 0" />
-            <geometry>
-                <mesh
-                    filename="package://vx01_description/meshes/drone/prop_link_0.STL" />
-            </geometry>
-        </collision>
+        <!-- Removed collision mesh for propeller to prevent physics instability (ODE Error) -->
     </link>
     <joint name="prop_0" type="continuous">

File: vx01_ws/src/vx01_description/urdf/drone/arm_1.xacro (robot description, xacro)
@@ -135,13 +135,5 @@
             </material>
         </visual>
-        <collision>
-            <origin
-                xyz="0 0 0"
-                rpy="0 0 0" />
-            <geometry>
-                <mesh
-                    filename="package://vx01_description/meshes/drone/prop_link_1.STL" />
-            </geometry>
-        </collision>
+        <!-- Removed collision mesh for propeller to prevent physics instability (ODE Error) -->
     </link>
     <joint name="prop_1" type="continuous">

File: vx01_ws/src/vx01_description/urdf/drone/arm_2.xacro (robot description, xacro)
@@ -135,13 +135,5 @@
             </material>
         </visual>
-        <collision>
-            <origin
-                xyz="0 0 0"
-                rpy="0 0 0" />
-            <geometry>
-                <mesh
-                    filename="package://vx01_description/meshes/drone/prop_link_2.STL" />
-            </geometry>
-        </collision>
+        <!-- Removed collision mesh for propeller to prevent physics instability (ODE Error) -->
     </link>
     <joint name="prop_2" type="continuous">

File: vx01_ws/src/vx01_description/urdf/drone/arm_3.xacro (robot description, xacro)
@@ -135,13 +135,5 @@
             </material>
         </visual>
-        <collision>
-            <origin
-                xyz="0 0 0"
-                rpy="0 0 0" />
-            <geometry>
-                <mesh
-                    filename="package://vx01_description/meshes/drone/prop_link_3.STL" />
-            </geometry>
-        </collision>
+        <!-- Removed collision mesh for propeller to prevent physics instability (ODE Error) -->
     </link>
     <joint name="prop_3" type="continuous">

Commit message: refactor: update propeller inertial properties, joint limits, and motor controller gains for improved stability

File: vx01_ws/src/vx01_description/urdf/drone/arm_0.xacro (robot description, xacro)
@@ -108,16 +108,13 @@
     <link name="prop_link_0">
         <inertial>
-            <origin
-                xyz="-4.0954E-08 -4.5858E-08 -0.0054488"
-                rpy="0 0 0" />
             <mass
-                value="0.0055592" />
+                value="0.02" />
             <inertia
-                ixx="6.7033E-06"
-                ixy="-9.2254E-06"
-                ixz="6.2283E-13"
-                iyy="1.3165E-05"
-                iyz="-4.5796E-13"
-                izz="1.983E-05" />
+                ixx="0.0001"
+                ixy="0.0"
+                ixz="0.0"
+                iyy="0.0001"
+                iyz="0.0"
+                izz="0.0001" />
         </inertial>
         <visual>
@@ -147,4 +144,5 @@
         <axis
             xyz="0 0 1" />
+        <limit effort="100.0" velocity="2000.0" />
     </joint>
 </robot>

File: vx01_ws/src/vx01_description/urdf/drone/arm_1.xacro (robot description, xacro)
@@ -108,16 +108,13 @@
     <link name="prop_link_1">
         <inertial>
-            <origin
-                xyz="-1.0522E-07 -6.9274E-08 -0.0054488"
-                rpy="0 0 0" />
             <mass
-                value="0.0055592" />
+                value="0.02" />
             <inertia
-                ixx="6.7033E-06"
-                ixy="-9.2254E-06"
-                ixz="3.8175E-13"
-                iyy="1.3165E-05"
-                iyz="1.2749E-12"
-                izz="1.983E-05" />
+                ixx="0.0001"
+                ixy="0.0"
+                ixz="0.0"
+                iyy="0.0001"
+                iyz="0.0"
+                izz="0.0001" />
         </inertial>
         <visual>
@@ -147,4 +144,5 @@
         <axis
             xyz="0 0 1" />
+        <limit effort="100.0" velocity="2000.0" />
     </joint>
 </robot>

File: vx01_ws/src/vx01_description/urdf/drone/arm_2.xacro (robot description, xacro)
@@ -108,16 +108,13 @@
     <link name="prop_link_2">
         <inertial>
-            <origin
-                xyz="4.0947E-08 4.5855E-08 -0.0054488"
-                rpy="0 0 0" />
             <mass
-                value="0.0055592" />
+                value="0.02" />
             <inertia
-                ixx="6.7032E-06"
-                ixy="-9.2253E-06"
-                ixz="-6.229E-13"
-                iyy="1.3165E-05"
-                iyz="4.5793E-13"
-                izz="1.983E-05" />
+                ixx="0.0001"
+                ixy="0.0"
+                ixz="0.0"
+                iyy="0.0001"
+                iyz="0.0"
+                izz="0.0001" />
         </inertial>
         <visual>
@@ -147,4 +144,5 @@
         <axis
             xyz="0 0 1" />
+        <limit effort="100.0" velocity="2000.0" />
     </joint>
 </robot>

File: vx01_ws/src/vx01_description/urdf/drone/arm_3.xacro (robot description, xacro)
@@ -108,16 +108,13 @@
     <link name="prop_link_3">
         <inertial>
-            <origin
-                xyz="-1.8711E-07 -1.6098E-07 -0.0054488"
-                rpy="0 0 0" />
             <mass
-                value="0.0055592" />
+                value="0.02" />
             <inertia
-                ixx="6.7033E-06"
-                ixy="-9.2254E-06"
-                ixz="1.6275E-12"
-                iyy="1.3165E-05"
-                iyz="3.5902E-13"
-                izz="1.983E-05" />
+                ixx="0.0001"
+                ixy="0.0"
+                ixz="0.0"
+                iyy="0.0001"
+                iyz="0.0"
+                izz="0.0001" />
         </inertial>
         <visual>
@@ -147,4 +144,5 @@
         <axis
             xyz="0 0 1" />
+        <limit effort="100.0" velocity="2000.0" />
     </joint>
 </robot>

File: vx01_ws/src/vx01_description/urdf/vx01.urdf.xacro (robot description, xacro)
@@ -66,5 +66,5 @@
                     <servo_max>2000</servo_max>
                     <type>VELOCITY</type>
-                    <p_gain>1.0</p_gain>
+                    <p_gain>10.0</p_gain>
                     <i_gain>0</i_gain>
                     <d_gain>0</d_gain>
@@ -81,5 +81,5 @@
                     <servo_max>2000</servo_max>
                     <type>VELOCITY</type>
-                    <p_gain>1.0</p_gain>
+                    <p_gain>10.0</p_gain>
                     <i_gain>0</i_gain>
                     <d_gain>0</d_gain>
@@ -96,5 +96,5 @@
                     <servo_max>2000</servo_max>
                     <type>VELOCITY</type>
-                    <p_gain>1.0</p_gain>
+                    <p_gain>10.0</p_gain>
                     <i_gain>0</i_gain>
                     <d_gain>0</d_gain>
@@ -111,5 +111,5 @@
                     <servo_max>2000</servo_max>
                     <type>VELOCITY</type>
-                    <p_gain>1.0</p_gain>
+                    <p_gain>10.0</p_gain>
                     <i_gain>0</i_gain>
                     <d_gain>0</d_gain>
