Commit message: changed controller for each leg

File: vx01_ws/src/vx01_description/urdf/base/base.xacro (robot description, xacro)
@@ -4,5 +4,5 @@
     <joint name="base_footprint_to_base_link" type="fixed">
         <origin
-            xyz="0 0 0.0528"
+            xyz="0 0 0"
             rpy="0 0 0" />
         <parent

File: vx01_ws/src/vx01_description/urdf/control/vx01.ros2_control.xacro (robot description, xacro)
@@ -10,6 +10,5 @@
         <ros2_control name="vx01_hardware" type="system">
             <hardware>
-                <plugin>gz_ros2_control/GazeboSimSystem</plugin>
-                <param name="position_proportional_gain">20.0</param>
+                <plugin>ign_ros2_control/IgnitionSystem</plugin>
             </hardware>
             <!-- ── Hexapod legs (18 joints) ── -->

File: vx01_ws/src/vx01_description/urdf/gazebo/vx01_sim.xacro (robot description, xacro)
@@ -317,4 +317,57 @@
         <selfCollide>false</selfCollide>
     </gazebo>
+    <!-- ── Drone Motors ─────────────────────────────────────────────────────── -->
+    <gazebo reference="motor_link_0">
+        <visual>
+            <material>
+                <ambient>0.25 0.25 0.25 1.0</ambient>
+                <diffuse>0.25 0.25 0.25 1.0</diffuse>
+                <specular>0.4 0.4 0.4 1.0</specular>
+                <emissive>0.0 0.0 0.0 1.0</emissive>
+            </material>
+        </visual>
+        <mu1>0.8</mu1>
+        <mu2>0.8</mu2>
+        <selfCollide>false</selfCollide>
+    </gazebo>
+    <gazebo reference="motor_link_1">
+        <visual>
+            <material>
+                <ambient>0.25 0.25 0.25 1.0</ambient>
+                <diffuse>0.25 0.25 0.25 1.0</diffuse>
+                <specular>0.4 0.4 0.4 1.0</specular>
+                <emissive>0.0 0.0 0.0 1.0</emissive>
+            </material>
+        </visual>
+        <mu1>0.8</mu1>
+        <mu2>0.8</mu2>
+        <selfCollide>false</selfCollide>
+    </gazebo>
+    <gazebo reference="motor_link_2">
+        <visual>
+            <material>
+                <ambient>0.25 0.25 0.25 1.0</ambient>
+                <diffuse>0.25 0.25 0.25 1.0</diffuse>
+                <specular>0.4 0.4 0.4 1.0</specular>
+                <emissive>0.0 0.0 0.0 1.0</emissive>
+            </material>
+        </visual>
+        <mu1>0.8</mu1>
+        <mu2>0.8</mu2>
+        <selfCollide>false</selfCollide>
+    </gazebo>
+    <gazebo reference="motor_link_3">
+        <visual>
+            <material>
+                <ambient>0.25 0.25 0.25 1.0</ambient>
+                <diffuse>0.25 0.25 0.25 1.0</diffuse>
+                <specular>0.4 0.4 0.4 1.0</specular>
+                <emissive>0.0 0.0 0.0 1.0</emissive>
+            </material>
+        </visual>
+        <mu1>0.8</mu1>
+        <mu2>0.8</mu2>
+        <selfCollide>false</selfCollide>
+    </gazebo>
     <!-- ── Propellers ─────────────────────────────────────────────────────── -->
     <gazebo reference="prop_link_0">

File: vx01_ws/src/vx01_description/urdf/vx01.urdf.xacro (robot description, xacro)
@@ -34,5 +34,5 @@
     <xacro:if value="${use_sim}">
         <gazebo>
-            <plugin filename="gz_ros2_control-system" name="gz_ros2_control::GazeboSimROS2ControlPlugin">
+            <plugin name="ign_ros2_control::IgnitionROS2ControlPlugin" filename="ign_ros2_control-system">
                 <parameters>$(find vx01_bringup)/config/vx01_controller_manager.yaml</parameters>
             </plugin>
