Commit message: fix(urdf): pass serial_port and baud_rate as xacro args instead of hardcoding

File: vx01_ws/src/vx01_description/urdf/vx01.urdf.xacro (robot description, xacro)
@@ -3,4 +3,8 @@
     <xacro:arg name="use_sim" default="false"/>
     <xacro:property name="use_sim" value="$(arg use_sim)"/>
+    <xacro:arg name="serial_port" default="/dev/ttyMAESTRO"/>
+    <xacro:property name="serial_port" value="$(arg serial_port)"/>
+    <xacro:arg name="baud_rate" default="115200"/>
+    <xacro:property name="baud_rate" value="$(arg baud_rate)"/>
     <!-- ── Base body ── -->
     <xacro:include filename="$(find vx01_description)/urdf/base/base.xacro"/>
@@ -27,6 +31,6 @@
     <xacro:vx01_ros2_control
         use_sim="${use_sim}"
-        serial_port="/dev/ttyACM0"
-        baud_rate="115200"
+        serial_port="${serial_port}"
+        baud_rate="${baud_rate}"
         pwm_frequency="50"
         gpio_chip="gpiochip0"/>

Commit message: feat: initialize backend node_modules and update robot URDF configuration

File: vx01_ws/src/vx01_description/urdf/vx01.urdf.xacro (robot description, xacro)
@@ -24,4 +24,8 @@
     <xacro:include filename="$(find vx01_description)/urdf/sensors/depth_camera.xacro"/>
     <xacro:include filename="$(find vx01_description)/urdf/sensors/imu.xacro"/>
+    <xacro:include filename="$(find vx01_description)/urdf/sensors/tf_mini.xacro"/>
+    <xacro:tf_mini parent="base_footprint">
+        <origin xyz="0 0 -0.05" rpy="0 1.5708 0"/>
+    </xacro:tf_mini>
     <!-- <xacro:include filename="$(find vx01_description)/urdf/sensors/tf_lidar.xacro"/> -->
     <!-- ROS2_control -->
